Commit message: feat(sim): 2단 트롤리 외형 + IMU/Depth카메라 + SLAM 실습 월드 + odom 보정
- robot_core: 박스 1개 → 2단 트롤리 외형(구동 베이스 + 모터4 + 프로파일
  프레임 + 선반 플레이트 + LCD). 치수 파라미터화, 무게중심 하향.
  바퀴를 차체 바깥으로 돌출시키고 모터를 베이스 하단에 배치.
- imu.xacro / depth_camera.xacro 추가 (gz imu, rgbd_camera 센서)
- bridge: 카메라 토픽 4종 + joint_states(바퀴 TF) 추가
- world: 단순 방 → 8x6m 실내(방3 + 복도 + 문3 + 장애물5), self-contained
  ground_plane 인라인화(외부 모델 의존 제거)
- launch_sim: gz 서버 미기동(-g) 수정, 스폰 -z 0.05(바퀴 지면 안착),
  복도 스폰 위치(-3,0)
- odom 보정: 4륜 스키드 회전 슬립 → wheel_separation 0.50→0.65(유효 트랙).
  IMU/ground-truth 비교로 회전·직진 ±2% 일치 검증.
- README: 시뮬 SLAM/Nav 실습 절차 + odom 재보정법 추가

Co-Authored-By: Claude Opus 4.8 (1M context) <noreply@anthropic.com>

File: tribo_description/urdf/gazebo_control.xacro (robot description, xacro)
@@ -8,6 +8,9 @@
         <right_joint>front_right_wheel_joint</right_joint>
         <right_joint>rear_right_wheel_joint</right_joint>
-        <!-- 실제 치수 -->
-        <wheel_separation>0.50</wheel_separation>
+        <!-- 물리 트랙은 0.50 (2*wheel_y) 이지만, 4륜 스키드 회전 슬립 보정을 위해 -->
+        <!-- 유효 트랙(effective)을 사용. odom(바퀴) 회전과 실제(IMU) 회전이 일치하도록 보정. -->
+        <!-- 검증 완료 - cmd wz 0.4/0.6/1.0 에서 odom/imu ratio = 1.0 ±2% (계통편차 없음) -->
+        <!-- 재보정 필요시 new = current * (odom 각속도 / imu 각속도) -->
+        <wheel_separation>0.65</wheel_separation>
         <wheel_radius>0.05</wheel_radius>
         <!-- ROS <-> GZ 브리지 토픽 -->

File: tribo_description/urdf/robot.urdf.xacro (robot description, xacro)
@@ -3,4 +3,6 @@
     <xacro:include filename="robot_core.xacro"/>
     <xacro:include filename="lidar.xacro" />
+    <xacro:include filename="imu.xacro" />
+    <xacro:include filename="depth_camera.xacro" />
     <xacro:include filename="robot_gazebo.xacro"/>
     <xacro:include filename="gazebo_control.xacro"/>

File: tribo_description/urdf/robot_core.xacro (robot description, xacro)
@@ -1,25 +1,83 @@
 <?xml version="1.0"?>
-    <robot name="tribo" xmlns:xacro="http://www.ros.org/wiki/xacro">
+<robot name="tribo" xmlns:xacro="http://www.ros.org/wiki/xacro">
     <xacro:include filename="inertial_macros.xacro"/>
+    <!-- ============================================================= -->
+    <!--  치수 파라미터 (단위 m)                                        -->
+    <!--  주의 - 모두 사진 비율로 추정한 값. 실측 확보 시 여기만 교체.  -->
+    <!--  좌표계 - X 전방, Y 좌측, Z 상방                               -->
+    <!--  base_link = 바퀴 축 평면(휠 중심 z=0)                         -->
+    <!-- ============================================================= -->
+    <!-- 바퀴 -->
+    <xacro:property name="wheel_radius" value="0.05"/>
+    <xacro:property name="wheel_width"  value="0.04"/>
+    <xacro:property name="wheel_x"      value="0.14"/>   <!-- 전후 휠 중심 (휠베이스/2) -->
+    <xacro:property name="wheel_y"      value="0.25"/>   <!-- 좌우 휠 중심 (트랙/2). 차체 반폭(0.21)보다 바깥 → 좌우 돌출 -->
+    <!-- 하단 베이스(구동부 박스). 좌우(Y)가 더 긴 직사각형 -->
+    <xacro:property name="base_x"       value="0.36"/>   <!-- 전후 길이 -->
+    <xacro:property name="base_y"       value="0.42"/>   <!-- 좌우 폭 -->
+    <xacro:property name="base_h"       value="0.12"/>   <!-- 높이 -->
+    <xacro:property name="base_bottom"  value="0.0"/>    <!-- 베이스 박스 바닥 z = 휠 축 높이. 모터/바퀴가 하단에 위치 -->
+    <xacro:property name="base_cz"      value="${base_bottom + base_h/2}"/>
+    <xacro:property name="deck_z"       value="${base_bottom + base_h}"/>  <!-- 베이스 상판 = 상단 프레임/라이다 기준면 -->
+    <!-- 상단 프레임(알루미늄 프로파일 케이지) -->
+    <xacro:property name="frame_h"      value="0.42"/>   <!-- 기둥 높이 -->
+    <xacro:property name="post_t"       value="0.02"/>   <!-- 프로파일 단면 -->
+    <xacro:property name="post_x"       value="0.15"/>   <!-- 기둥 X 위치 -->
+    <xacro:property name="post_y"       value="0.18"/>   <!-- 기둥 Y 위치 (차체 안쪽) -->
+    <xacro:property name="top_z"        value="${deck_z + frame_h}"/>  <!-- 상단 프레임 z -->
+    <!-- 라이다(하단 상판 전방 중앙) -->
+    <xacro:property name="lidar_x"      value="0.16"/>
     <!-- Materials -->
-    <material name="white"><color rgba="1 1 1 1"/></material>
+    <material name="white"><color rgba="0.9 0.9 0.9 1"/></material>
     <material name="orange"><color rgba="1 0.3 0.1 1"/></material>
     <material name="blue"><color rgba="0.2 0.2 1 1"/></material>
-    <material name="black"><color rgba="0 0 0 1"/></material>
-    <!-- BASE LINK -->
+    <material name="black"><color rgba="0.05 0.05 0.05 1"/></material>
+    <material name="red"><color rgba="0.9 0.3 0.25 1"/></material>
+    <material name="silver"><color rgba="0.75 0.75 0.78 1"/></material>
+    <material name="cyan"><color rgba="0.2 0.6 0.7 1"/></material>
+    <material name="green"><color rgba="0.1 0.8 0.2 1"/></material>
+    <!-- ============================================================= -->
+    <!--  BASE LINK                                                     -->
+    <!-- ============================================================= -->
     <link name="base_link"/>
-    <!-- CHASSIS -->
+    <!-- ============================================================= -->
+    <!--  CHASSIS = 하단 구동 베이스 (박스 + 모터 하우징 비주얼)        -->
+    <!-- ============================================================= -->
     <link name="chassis">
-        <visual>
-            <origin xyz="0 0 0.075"/>
-            <geometry><box size="0.30 0.50 0.10"/></geometry>
+        <!-- 베이스 박스 -->
+        <visual>
+            <origin xyz="0 0 ${base_cz}"/>
+            <geometry><box size="${base_x} ${base_y} ${base_h}"/></geometry>
             <material name="white"/>
         </visual>
         <collision>
-            <origin xyz="0 0 0.075"/>
-            <geometry><box size="0.30 0.50 0.10"/></geometry>
-        </collision>
-        <xacro:inertial_box mass="0.4" x="0.30" y="0.50" z="0.10">
-        <origin xyz="0 0 0.075" rpy="0 0 0"/>
+            <origin xyz="0 0 ${base_cz}"/>
+            <geometry><box size="${base_x} ${base_y} ${base_h}"/></geometry>
+        </collision>
+        <!-- 모터 하우징 4개 (빨간 원통). 베이스 하단(z=0)에 부착, 바퀴 안쪽 -->
+        <!-- 모터(y≈±0.19)보다 바퀴(y=±0.25)가 바깥 → 좌우로 돌출 -->
+        <visual>
+            <origin xyz="${wheel_x} ${wheel_y - 0.06} 0" rpy="${pi/2} 0 0"/>
+            <geometry><cylinder radius="0.04" length="0.08"/></geometry>
+            <material name="red"/>
+        </visual>
+        <visual>
+            <origin xyz="${wheel_x} ${-(wheel_y - 0.06)} 0" rpy="${pi/2} 0 0"/>
+            <geometry><cylinder radius="0.04" length="0.08"/></geometry>
+            <material name="red"/>
+        </visual>
+        <visual>
+            <origin xyz="${-wheel_x} ${wheel_y - 0.06} 0" rpy="${pi/2} 0 0"/>
+            <geometry><cylinder radius="0.04" length="0.08"/></geometry>
+            <material name="red"/>
+        </visual>
+        <visual>
+            <origin xyz="${-wheel_x} ${-(wheel_y - 0.06)} 0" rpy="${pi/2} 0 0"/>
+            <geometry><cylinder radius="0.04" length="0.08"/></geometry>
+            <material name="red"/>
+        </visual>
+        <!-- 무게 중심을 낮게 두기 위해 베이스에 질량 집중 -->
+        <xacro:inertial_box mass="3.0" x="${base_x}" y="${base_y}" z="${base_h}">
+            <origin xyz="0 0 ${base_cz}" rpy="0 0 0"/>
         </xacro:inertial_box>
     </link>
@@ -29,14 +87,17 @@
         <origin xyz="0 0 0"/>
     </joint>
+    <!-- ============================================================= -->
+    <!--  바퀴 4개 (좌측 axis +Z, 우측 axis -Z) — 기존 구조 유지        -->
+    <!-- ============================================================= -->
     <!-- FRONT LEFT -->
     <link name="front_left_wheel">
         <visual>
-            <geometry><cylinder radius="0.05" length="0.04"/></geometry>
-            <material name="blue"/>
-        </visual>
-        <collision>
-            <geometry><cylinder radius="0.05" length="0.04"/></geometry>
-        </collision>
-        <xacro:inertial_cylinder mass="0.1" length="0.04" radius="0.05">
+            <geometry><cylinder radius="${wheel_radius}" length="${wheel_width}"/></geometry>
+            <material name="black"/>
+        </visual>
+        <collision>
+            <geometry><cylinder radius="${wheel_radius}" length="${wheel_width}"/></geometry>
+        </collision>
+        <xacro:inertial_cylinder mass="0.1" length="${wheel_width}" radius="${wheel_radius}">
             <origin xyz="0 0 0" rpy="0 0 0"/>
         </xacro:inertial_cylinder>
@@ -45,6 +106,5 @@
         <parent link="base_link"/>
         <child  link="front_left_wheel"/>
-        <!-- x = +0.095, y = +0.1075 -->
-        <origin xyz="0.10 0.25 0" rpy="-${pi/2} 0 0"/>
+        <origin xyz="${wheel_x} ${wheel_y} 0" rpy="-${pi/2} 0 0"/>
         <axis xyz="0 0 1"/>
     </joint>
@@ -52,11 +112,11 @@
     <link name="front_right_wheel">
         <visual>
-            <geometry><cylinder radius="0.05" length="0.04"/></geometry>
-            <material name="blue"/>
-        </visual>
-        <collision>
-            <geometry><cylinder radius="0.05" length="0.04"/></geometry>
-        </collision>
-        <xacro:inertial_cylinder mass="0.1" length="0.04" radius="0.05">
+            <geometry><cylinder radius="${wheel_radius}" length="${wheel_width}"/></geometry>
+            <material name="black"/>
+        </visual>
+        <collision>
+            <geometry><cylinder radius="${wheel_radius}" length="${wheel_width}"/></geometry>
+        </collision>
+        <xacro:inertial_cylinder mass="0.1" length="${wheel_width}" radius="${wheel_radius}">
             <origin xyz="0 0 0" rpy="0 0 0"/>
         </xacro:inertial_cylinder>
@@ -65,6 +125,5 @@
         <parent link="base_link"/>
         <child  link="front_right_wheel"/>
-        <!-- x = +0.095, y = -0.1075 -->
-        <origin xyz="0.10 -0.25 0" rpy="${pi/2} 0 0"/>
+        <origin xyz="${wheel_x} ${-wheel_y} 0" rpy="${pi/2} 0 0"/>
         <axis xyz="0 0 -1"/>
     </joint>
@@ -72,11 +131,11 @@
     <link name="rear_left_wheel">
         <visual>
-            <geometry><cylinder radius="0.05" length="0.04"/></geometry>
-            <material name="blue"/>
-        </visual>
-        <collision>
-            <geometry><cylinder radius="0.05" length="0.04"/></geometry>
-        </collision>
-        <xacro:inertial_cylinder mass="0.1" length="0.04" radius="0.05">
+            <geometry><cylinder radius="${wheel_radius}" length="${wheel_width}"/></geometry>
+            <material name="black"/>
+        </visual>
+        <collision>
+            <geometry><cylinder radius="${wheel_radius}" length="${wheel_width}"/></geometry>
+        </collision>
+        <xacro:inertial_cylinder mass="0.1" length="${wheel_width}" radius="${wheel_radius}">
             <origin xyz="0 0 0" rpy="0 0 0"/>
         </xacro:inertial_cylinder>
@@ -85,6 +144,5 @@
         <parent link="base_link"/>
         <child  link="rear_left_wheel"/>
-        <!-- x = -0.095, y = +0.1075 -->
-        <origin xyz="-0.10 0.25 0" rpy="-${pi/2} 0 0"/>
+        <origin xyz="${-wheel_x} ${wheel_y} 0" rpy="-${pi/2} 0 0"/>
         <axis xyz="0 0 1"/>
     </joint>
@@ -92,11 +150,11 @@
     <link name="rear_right_wheel">
         <visual>
-            <geometry><cylinder radius="0.05" length="0.04"/></geometry>
-            <material name="blue"/>
-        </visual>
-        <collision>
-            <geometry><cylinder radius="0.05" length="0.04"/></geometry>
-        </collision>
-        <xacro:inertial_cylinder mass="0.1" length="0.04" radius="0.05">
+            <geometry><cylinder radius="${wheel_radius}" length="${wheel_width}"/></geometry>
+            <material name="black"/>
+        </visual>
+        <collision>
+            <geometry><cylinder radius="${wheel_radius}" length="${wheel_width}"/></geometry>
+        </collision>
+        <xacro:inertial_cylinder mass="0.1" length="${wheel_width}" radius="${wheel_radius}">
             <origin xyz="0 0 0" rpy="0 0 0"/>
         </xacro:inertial_cylinder>
@@ -105,55 +163,151 @@
         <parent link="base_link"/>
         <child  link="rear_right_wheel"/>
-        <!-- x = -0.095, y = -0.1075 -->
-        <origin xyz="-0.10 -0.25 0" rpy="${pi/2} 0 0"/>
+        <origin xyz="${-wheel_x} ${-wheel_y} 0" rpy="${pi/2} 0 0"/>
         <axis xyz="0 0 -1"/>
     </joint>
+    <!-- ============================================================= -->
+    <!--  상단 프레임 케이지 (기둥 4 + 상단 레일 4 + 디스플레이 + 버튼) -->
+    <!--  단일 fixed 링크로 묶음. 좌표는 base_link 기준.               -->
+    <!-- ============================================================= -->
+    <link name="frame">
+        <!-- 수직 기둥 4개 -->
+        <visual>
+            <origin xyz="${post_x} ${post_y} ${deck_z + frame_h/2}"/>
+            <geometry><box size="${post_t} ${post_t} ${frame_h}"/></geometry>
+            <material name="silver"/>
+        </visual>
+        <visual>
+            <origin xyz="${post_x} ${-post_y} ${deck_z + frame_h/2}"/>
+            <geometry><box size="${post_t} ${post_t} ${frame_h}"/></geometry>
+            <material name="silver"/>
+        </visual>
+        <visual>
+            <origin xyz="${-post_x} ${post_y} ${deck_z + frame_h/2}"/>
+            <geometry><box size="${post_t} ${post_t} ${frame_h}"/></geometry>
+            <material name="silver"/>
+        </visual>
+        <visual>
+            <origin xyz="${-post_x} ${-post_y} ${deck_z + frame_h/2}"/>
+            <geometry><box size="${post_t} ${post_t} ${frame_h}"/></geometry>
+            <material name="silver"/>
+        </visual>
+        <!-- 상단 레일 X 방향 2개 -->
+        <visual>
+            <origin xyz="0 ${post_y} ${top_z}"/>
+            <geometry><box size="${2*post_x + post_t} ${post_t} ${post_t}"/></geometry>
+            <material name="silver"/>
+        </visual>
+        <visual>
+            <origin xyz="0 ${-post_y} ${top_z}"/>
+            <geometry><box size="${2*post_x + post_t} ${post_t} ${post_t}"/></geometry>
+            <material name="silver"/>
+        </visual>
+        <!-- 상단 레일 Y 방향 2개 -->
+        <visual>
+            <origin xyz="${post_x} 0 ${top_z}"/>
+            <geometry><box size="${post_t} ${2*post_y} ${post_t}"/></geometry>
+            <material name="silver"/>
+        </visual>
+        <visual>
+            <origin xyz="${-post_x} 0 ${top_z}"/>
+            <geometry><box size="${post_t} ${2*post_y} ${post_t}"/></geometry>
+            <material name="silver"/>
+        </visual>
+        <!-- 선반 플레이트 (프레임 기둥에 끼워진 중상단 선반. 지붕 아님) -->
+        <visual>
+            <origin xyz="0 0 ${deck_z + 0.28}"/>
+            <geometry><box size="${2*post_x + post_t} ${2*post_y + post_t} 0.02"/></geometry>
+            <material name="white"/>
+        </visual>
+        <collision>
+            <origin xyz="0 0 ${deck_z + 0.28}"/>
+            <geometry><box size="${2*post_x + post_t} ${2*post_y + post_t} 0.02"/></geometry>
+        </collision>
+        <!-- 전면 가로 프로파일 2개 (LCD/카메라 장착용) -->
+        <visual>
+            <origin xyz="${post_x} 0 ${deck_z + 0.18}"/>
+            <geometry><box size="${post_t} ${2*post_y} ${post_t}"/></geometry>
+            <material name="silver"/>
+        </visual>
+        <visual>
+            <origin xyz="${post_x} 0 ${deck_z + 0.32}"/>
+            <geometry><box size="${post_t} ${2*post_y} ${post_t}"/></geometry>
+            <material name="silver"/>
+        </visual>
+        <!-- 디스플레이 (전면 가로바에 부착) -->
+        <visual>
+            <origin xyz="${post_x + 0.012} 0 ${deck_z + 0.18}"/>
+            <geometry><box size="0.02 0.24 0.14"/></geometry>
+            <material name="cyan"/>
+        </visual>
+        <!-- 전원 버튼 (녹색, 가로바에 부착) -->
+        <visual>
+            <origin xyz="${post_x + 0.012} 0.14 ${deck_z + 0.32}"/>
+            <geometry><box size="0.03 0.03 0.03"/></geometry>
+            <material name="green"/>
+        </visual>
+        <!-- 충돌은 기둥만 (프레임 물리 외곽) -->
+        <collision>
+            <origin xyz="${post_x} ${post_y} ${deck_z + frame_h/2}"/>
+            <geometry><box size="${post_t} ${post_t} ${frame_h}"/></geometry>
+        </collision>
+        <collision>
+            <origin xyz="${post_x} ${-post_y} ${deck_z + frame_h/2}"/>
+            <geometry><box size="${post_t} ${post_t} ${frame_h}"/></geometry>
+        </collision>
+        <collision>
+            <origin xyz="${-post_x} ${post_y} ${deck_z + frame_h/2}"/>
+            <geometry><box size="${post_t} ${post_t} ${frame_h}"/></geometry>
+        </collision>
+        <collision>
+            <origin xyz="${-post_x} ${-post_y} ${deck_z + frame_h/2}"/>
+            <geometry><box size="${post_t} ${post_t} ${frame_h}"/></geometry>
+        </collision>
+        <!-- 프레임 전체 질량 근사 (기둥 + 레일 + 2층 판) -->
+        <xacro:inertial_box mass="1.2" x="${2*post_x}" y="${2*post_y}" z="${frame_h}">
+            <origin xyz="0 0 ${deck_z + frame_h/2}" rpy="0 0 0"/>
+        </xacro:inertial_box>
+    </link>
+    <joint name="frame_joint" type="fixed">
+        <parent link="chassis"/>
+        <child  link="frame"/>
+        <origin xyz="0 0 0"/>
+    </joint>
+    <!-- ============================================================= -->
+    <!--  라이다 (하단 상판 전방 중앙)                                  -->
+    <!-- ============================================================= -->
     <link name="lidar_mount">
         <visual>
-            <origin xyz="0 0 0" rpy="0 0 0"/>
-            <geometry>
-                <cylinder radius="0.025" length="0.02"/>
-            </geometry>
-            <material name="black">
-                <color rgba="0 0 0 1"/>
-            </material>
-        </visual>
-        <collision>
-            <origin xyz="0 0 0" rpy="0 0 0"/>
-            <geometry>
-                <cylinder radius="0.025" length="0.02"/>
-            </geometry>
+            <origin xyz="0 0 0.01" rpy="0 0 0"/>
+            <geometry><cylinder radius="0.025" length="0.02"/></geometry>
+            <material name="black"/>
+        </visual>
+        <collision>
+            <origin xyz="0 0 0.01" rpy="0 0 0"/>
+            <geometry><cylinder radius="0.025" length="0.02"/></geometry>
         </collision>
         <inertial>
-            <origin xyz="0 0 0" rpy="0 0 0"/>
+            <origin xyz="0 0 0.01" rpy="0 0 0"/>
             <mass value="0.05"/>
-            <!-- 대략적인 관성치 m*r^2/2, m*(3r^2+h^2)/12 등 근사 -->
             <inertia ixx="3.0e-05" ixy="0" ixz="0" iyy="3.0e-05" iyz="0" izz="3.0e-05"/>
         </inertial>
     </link>
-    <!-- 마운트를 섀시에 고정 -->
     <joint name="lidar_mount_fixed_joint" type="fixed">
         <parent link="chassis"/>
         <child link="lidar_mount"/>
-        <!-- 섀시 위쪽 중앙에 배치. 필요시 xyz 조정 -->
-        <origin xyz="0.1 0.0 0.125" rpy="0 0 0"/>
-    </joint>
-    <!-- 레이저 링크 라이다 본체를 단순 실린더로 표현 -->
+        <!-- 하단 베이스 상판 전방 중앙 -->
+        <origin xyz="${lidar_x} 0.0 ${deck_z}" rpy="0 0 0"/>
+    </joint>
+    <!-- 레이저 링크 (라이다 본체). yaw=π 는 실로봇 거꾸로 마운트 보정값 -->
+    <!-- ⚠ 새 마운트 방향은 실로봇에서 재검증 필요 -->
     <link name="laser_link">
         <visual>
             <origin xyz="0 0 0" rpy="0 0 0"/>
-            <geometry>
-            <!-- 지름 약 6cm, 높이 6cm 정도의 라이다로 가정 -->
-                <cylinder radius="0.03" length="0.06"/>
-            </geometry>
-            <material name="blue">
-                <color rgba="0.2 0.2 1 1"/>
-            </material>
-        </visual>
-        <collision>
-            <origin xyz="0 0 0" rpy="0 0 0"/>
-            <geometry>
-                <cylinder radius="0.03" length="0.06"/>
-            </geometry>
+            <geometry><cylinder radius="0.03" length="0.06"/></geometry>
+            <material name="blue"/>
+        </visual>
+        <collision>
+            <origin xyz="0 0 0" rpy="0 0 0"/>
+            <geometry><cylinder radius="0.03" length="0.06"/></geometry>
         </collision>
         <inertial>
@@ -163,9 +317,60 @@
         </inertial>
     </link>
-    <!-- 레이저를 마운트 위에 고정. 라이다가 거꾸로 마운트되어 있어 yaw=π로 보정 -->
     <joint name="laser_link_fixed_joint" type="fixed">
-    <parent link="lidar_mount"/>
-    <child link="laser_link"/>
-    <origin xyz="0.0 0.0 0.05" rpy="0 0 ${pi}"/>
+        <parent link="lidar_mount"/>
+        <child link="laser_link"/>
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