Commit message: refactor: IMU·EKF 완전 제거, 휠 오도메트리 단일 경로로 전환
이 기체 보드 IMU 는 yaw 를 만들 두 경로가 모두 고장이다: 절대 yaw(orientation)
는 펌웨어가 갱신 안 하고(freeze), 대안인 자이로(gz)는 지속 회전 약 2.4초(≈24°)
후 0 으로 죽는다. 라이다 독립 측정(스캔 상관)으로 실제 회전 +133°, 휠 +126°(5%
일치)인데 IMU 적분만 +24°에서 멈추는 것을 확인. EKF 는 yaw 를 IMU 자이로로만
추정하므로 회전 중 /odom yaw 가 멈춰 map building 이 깨졌다. 휠·라이다가 일치
하므로 휠 오도메트리만으로 충분 → IMU·EKF 를 ws 전체에서 제거.

실로봇:
- bringup.launch.py: use_ekf/ekf_node/odom_node_with_ekf 제거. odom_publisher
  가 /odom + TF(odom->base_link) 직접 발행하는 단일 경로로. track_width 0.838 고정.
- param/ekf.yaml 삭제, package.xml 에서 robot_localization 의존성 제거.
- bringup.py: IMU 파라미터/퍼블리셔/타이머/_imu_timer_cb/_euler_to_quat 제거.
- config/bringup.yaml: IMU 블록 제거.

odom 도구:
- rotation_calib.py 삭제(IMU 기준값 의존 → 무력화) + entry point 제거.
  track_width 재조정은 이제 라이다 스캔 상관으로 실제 회전각을 재는 수동 절차.
- odom_source.py 삭제(orphaned, /imu/data_raw 구독).

sim(gazebo):
- imu.xacro 삭제 + include 제거, robot_core.xacro imu_link/joint 제거,
  world 2개 gz-sim-imu-system 플러그인 제거, bridge imu 항목 제거.

기타:
- ekf_localization.yaml 삭제(orphaned). README 의 IMU/EKF/rotation_calib 서술 정리.
- (동봉) 이전 세션의 pwm_max_percent 파라미터(default 100.0 = 무동작)가
  bringup.py/yaml 에 함께 반영됨.

검증: PC colcon build 성공(robot_localization 없이), launch 구성 Node 4개
(ekf_node 없음, odom_publisher 단일), xacro/world XML 유효. 로봇 실동작은
로봇 재기동 시 확인 예정.

Co-Authored-By: Claude Opus 4.8 (1M context) <noreply@anthropic.com>

File: tribo_description/urdf/gazebo_control.xacro (robot description, xacro)
@@ -9,7 +9,7 @@
         <right_joint>rear_right_wheel_joint</right_joint>
         <!-- 물리 트랙은 0.50 (2*wheel_y) 이지만, 4륜 스키드 회전 슬립 보정을 위해 -->
-        <!-- 유효 트랙(effective)을 사용. odom(바퀴) 회전과 실제(IMU) 회전이 일치하도록 보정. -->
-        <!-- 검증 완료 - cmd wz 0.4/0.6/1.0 에서 odom/imu ratio = 1.0 ±2% (계통편차 없음) -->
-        <!-- 재보정 필요시 new = current * (odom 각속도 / imu 각속도) -->
+        <!-- 유효 트랙(effective)을 사용해 odom(바퀴) 회전이 실제 회전과 일치하도록 보정. -->
+        <!-- cmd wz 0.4/0.6/1.0 에서 회전 ratio 1.0 ±2% 검증(계통편차 없음). -->
+        <!-- 재보정 필요시 라이다 스캔으로 실제 회전각을 재어 new = current * (odom/실제). -->
         <wheel_separation>0.65</wheel_separation>
         <wheel_radius>0.05</wheel_radius>

File: tribo_description/urdf/robot.urdf.xacro (robot description, xacro)
@@ -3,5 +3,4 @@
     <xacro:include filename="robot_core.xacro"/>
     <xacro:include filename="lidar.xacro" />
-    <xacro:include filename="imu.xacro" />
     <xacro:include filename="depth_camera.xacro" />
     <xacro:include filename="robot_gazebo.xacro"/>

File: tribo_description/urdf/robot_core.xacro (robot description, xacro)
@@ -323,24 +323,4 @@
     </joint>
     <!-- ============================================================= -->
-    <!--  IMU (베이스 중앙)                                             -->
-    <!-- ============================================================= -->
-    <link name="imu_link">
-        <visual>
-            <origin xyz="0 0 0" rpy="0 0 0"/>
-            <geometry><box size="0.02 0.02 0.01"/></geometry>
-            <material name="orange"/>
-        </visual>
-        <inertial>
-            <origin xyz="0 0 0" rpy="0 0 0"/>
-            <mass value="0.01"/>
-            <inertia ixx="1.0e-06" ixy="0" ixz="0" iyy="1.0e-06" iyz="0" izz="1.0e-06"/>
-        </inertial>
-    </link>
-    <joint name="imu_joint" type="fixed">
-        <parent link="chassis"/>
-        <child link="imu_link"/>
-        <origin xyz="0 0 ${deck_z}" rpy="0 0 0"/>
-    </joint>
-    <!-- ============================================================= -->
     <!--  Depth 카메라 (상단 프레임 전면, 전방 주시)                    -->
     <!-- ============================================================= -->
