Commit message: feat: invert lidar URDF mount + auto-fullscreen RViz on robot LCD
- URDF: laser_link_fixed_joint yaw set to pi to compensate for the
  upside-down LiDAR mount so /scan frame aligns with the environment.
- tribo_navigation/bringup_launch.xml: add use_rviz arg (default true)
  and an RViz node that runs through launch_rviz_on_lcd.sh, which
  resolves DISPLAY/XAUTHORITY on the robots GNOME Wayland session and
  starts rviz2 --fullscreen on the connected LCD.
- scripts/launch_rviz_on_lcd.sh: new wrapper for runtime env assembly.
- setup.py: install scripts/*.sh into lib/<pkg>/ so the launch can
  locate the wrapper.
- README 6-4: LCD auto-display notes + PC simultaneous view tip.

Co-Authored-By: Claude Opus 4.7 (1M context) <noreply@anthropic.com>

File: tribo_description/urdf/robot_core.xacro (robot description, xacro)
@@ -163,9 +163,9 @@
         </inertial>
     </link>
-    <!-- 레이저를 마운트 위에 고정 -->
+    <!-- 레이저를 마운트 위에 고정. 라이다가 거꾸로 마운트되어 있어 yaw=π로 보정 -->
     <joint name="laser_link_fixed_joint" type="fixed">
     <parent link="lidar_mount"/>
     <child link="laser_link"/>
-    <origin xyz="0.0 0.0 0.05" rpy="0 0 0"/>
+    <origin xyz="0.0 0.0 0.05" rpy="0 0 ${pi}"/>
     </joint>
 </robot>

Commit message: fix(geom): 구조 변경 + 100mm 메카넘 실측 재캘리브 (기체 7b6a)
줄자 실측:
- 물리 track 0.71 -> 0.74 (좌우 바퀴 중심-중심)
- 휠베이스 0.40 (신규 기록)

지상 직진 캘리브로 wheel_radius 0.0430 -> 0.0563:
- 2.8m 주행, 휠 경로(ticks) vs 실측 경로 비교. 활주 ~5cm 보정.
- 2.5m 주행(m2 고장 상태)과 2.8m 주행(정비 후)의 ticks/m 이
  12222 vs 12141 로 0.7% 차이뿐이라 두 측정이 서로를 검증한다.
- 공칭 0.050 대비 x1.125 로, 이 기체가 고무바퀴 시절 쓰던 x1.121 과
  거의 일치한다. 보정계수가 바퀴가 아니라 기체(ticks_per_rev/기어비)에
  붙어 있다는 기존 해석과 맞는다.

⚠️ 1차 측정(1.13m)은 x1.244 라는 물리적으로 불가능한 값을 줬다.
   유효반경이 물리반경보다 클 수 없다. 기준점 오차로 보고 버렸고,
   거리를 2.5m 이상으로 늘리자 값이 수렴했다. 짧은 거리 측정은 쓰지 말 것.

robot_core.xacro 의 wheel_x/wheel_y 는 파일 주석대로 사진 비율 추정치였고
실측(0.28/0.50)과 크게 어긋나 있었다. 0.20/0.37 로 교체.

Co-Authored-By: Claude Opus 5 (1M context) <noreply@anthropic.com>

File: tribo_description/urdf/robot_core.xacro (robot description, xacro)
@@ -9,11 +9,15 @@
     <!-- ============================================================= -->
     <!-- 바퀴 -->
+    <!-- 100mm 메카넘 공칭 반경. 운동학용 보정 반경(robot_geom.yaml 의 wheel_radius)과 -->
+    <!-- 는 성격이 다르다. 여기는 물리 형상이므로 공칭값을 쓴다. -->
     <xacro:property name="wheel_radius" value="0.05"/>
     <xacro:property name="wheel_width"  value="0.04"/>
-    <xacro:property name="wheel_x"      value="0.14"/>   <!-- 전후 휠 중심 (휠베이스/2) -->
-    <xacro:property name="wheel_y"      value="0.25"/>   <!-- 좌우 휠 중심 (트랙/2). 차체 반폭(0.21)보다 바깥 → 좌우 돌출 -->
+    <!-- 2026-08-19 실측으로 교체. 기존 0.14/0.25 는 위 주석대로 사진 비율 추정치였고 -->
+    <!-- 실측(휠베이스 0.40, 트랙 0.74)과 크게 어긋나 있었다. -->
+    <xacro:property name="wheel_x"      value="0.20"/>   <!-- 전후 휠 중심 (휠베이스 0.40 의 절반) -->
+    <xacro:property name="wheel_y"      value="0.37"/>   <!-- 좌우 휠 중심 (트랙 0.74 의 절반). 차체 반폭(0.21)보다 16cm 바깥 → 좌우 크게 돌출 -->
     <!-- 하단 베이스(구동부 박스). 좌우(Y)가 더 긴 직사각형 -->
     <xacro:property name="base_x"       value="0.36"/>   <!-- 전후 길이 -->
-    <xacro:property name="base_y"       value="0.42"/>   <!-- 좌우 폭 -->
+    <xacro:property name="base_y"       value="0.42"/>   <!-- 좌우 폭. ⚠️ 미실측 추정치 — 구조 변경분 반영 안 됨 -->
     <xacro:property name="base_h"       value="0.12"/>   <!-- 높이 -->
     <xacro:property name="base_bottom"  value="0.0"/>    <!-- 베이스 박스 바닥 z = 휠 축 높이. 모터/바퀴가 하단에 위치 -->

Commit message: fix(description): 차체 치수를 바퀴 실측 기하에서 유도한다
Gazebo 에서 모터가 차체와 떨어져 떠 보였다. 원인은 휠베이스(0.40)가 차체
전후 길이(0.36)보다 길어 모터 축이 아예 차체 밖에 있었던 것이다. base_y
0.42 도 "미실측 추정치" 로 표시된 채 구조 변경분이 반영되지 않고 있었다.

숫자를 베껴 적는 대신 바퀴 실측 기하에서 유도하도록 바꿨다.
  base_x = 2*(wheel_x + wheel_radius)      = 0.50
  base_y = 2*(wheel_y - wheel_width/2)     = 0.70
전폭은 바퀴 안쪽 면까지만 잡는다. footprint 전폭 0.78 을 그대로 쓰면 바퀴가
박스에 파묻히기 때문이다. 이제 바퀴 4개가 차체 밖으로 40 mm 온전히 드러난다.
프레임 기둥도 frame_inset 기준 유도식으로 바꿔 차체 크기를 따라가게 했고,
모터는 바퀴 축 위 바퀴 안쪽 면에 직결했다.

로봇 전체 외곽은 0.50 x 0.78 로 nav2 footprint 와 그대로 일치한다.

작업 중 센서 TF 가 프레임 모델에 딸려 움직이는 회귀를 발견해 함께 고쳤다.
camera_joint 의 x 가 ${post_x + 0.02} 였던 탓에, 기둥 위치를 유도식으로 바꾸자
실물 카메라는 그대로인데 TF 만 0.17 -> 0.22 로 5 cm 밀렸다. 프레임 치수는
아직 미실측 추정치라 여기에 센서를 묶으면 모델을 손볼 때마다 실로봇 TF 가
흔들린다. camera_x(0.17) 프로퍼티를 따로 두어 원래 값으로 되돌리고, lidar_x
와 함께 "센서 장착 위치는 차체/프레임 모델에 묶지 않는다" 는 규칙을 주석으로
남겼다. 프레임 가로바가 이보다 조금 앞이라 비주얼상 7 mm 떠 보이지만 TF
안정성을 우선했다.

TF 영향 - 없다. HEAD 로 생성한 URDF 와 조인트 10개를 타입/parent/child 와
원점 xyz/rpy 까지 수치 비교했고, 전체 최대 편차가 2.8e-17 m 다. 그마저도
camera_joint 에서 0.17 리터럴과 0.15+0.02 부동소수 표기가 갈린 것뿐이라
물리적으로 0 이고, 나머지 9개는 정확히 0 이다. 즉 이 커밋은 visual /
collision / inertial 만 바꾸며 실로봇 주행에 영향이 없다.

xacro 파싱과 robot_description YAML 로드는 통과 확인했다.

Co-Authored-By: Claude Opus 5 (1M context) <noreply@anthropic.com>

File: tribo_description/urdf/robot_core.xacro (robot description, xacro)
@@ -17,7 +17,17 @@
     <xacro:property name="wheel_x"      value="0.20"/>   <!-- 전후 휠 중심 (휠베이스 0.40 의 절반) -->
     <xacro:property name="wheel_y"      value="0.37"/>   <!-- 좌우 휠 중심 (트랙 0.74 의 절반). 차체 반폭(0.21)보다 16cm 바깥 → 좌우 크게 돌출 -->
-    <!-- 하단 베이스(구동부 박스). 좌우(Y)가 더 긴 직사각형 -->
-    <xacro:property name="base_x"       value="0.36"/>   <!-- 전후 길이 -->
-    <xacro:property name="base_y"       value="0.42"/>   <!-- 좌우 폭. ⚠️ 미실측 추정치 — 구조 변경분 반영 안 됨 -->
+    <!-- ============================================================= -->
+    <!--  하단 베이스(구동부 박스)                                       -->
+    <!--  전장(X)은 nav2 실측 footprint 그대로. 같은 실측 기하에서       -->
+    <!--  유도하며 숫자를 베껴 적지 않는다.                              -->
+    <!--    전장 0.50 = 2*(휠베이스/2 + 바퀴반경)  = footprint X 와 동일  -->
+    <!--  전폭(Y)은 바퀴 안쪽 면까지만 잡는다. footprint 전폭 0.78 은     -->
+    <!--  바퀴 바깥면까지의 값이라 그대로 쓰면 바퀴가 박스에 파묻힌다.    -->
+    <!--    전폭 0.70 = 2*(트랙/2 - 바퀴폭/2)                            -->
+    <!--  → 바퀴 4개가 박스 밖으로 온전히 드러난다.                      -->
+    <!--  로봇 전체 외곽은 여전히 0.50 x 0.78 = nav2 footprint 그대로다. -->
+    <!-- ============================================================= -->
+    <xacro:property name="base_x"       value="${2*(wheel_x + wheel_radius)}"/>   <!-- 전장 0.50 -->
+    <xacro:property name="base_y"       value="${2*(wheel_y - wheel_width/2)}"/>  <!-- 전폭 0.70 -->
     <xacro:property name="base_h"       value="0.12"/>   <!-- 높이 -->
     <xacro:property name="base_bottom"  value="0.0"/>    <!-- 베이스 박스 바닥 z = 휠 축 높이. 모터/바퀴가 하단에 위치 -->
@@ -27,9 +37,29 @@
     <xacro:property name="frame_h"      value="0.42"/>   <!-- 기둥 높이 -->
     <xacro:property name="post_t"       value="0.02"/>   <!-- 프로파일 단면 -->
-    <xacro:property name="post_x"       value="0.15"/>   <!-- 기둥 X 위치 -->
-    <xacro:property name="post_y"       value="0.18"/>   <!-- 기둥 Y 위치 (차체 안쪽) -->
+    <!-- 기둥은 차체 모서리에서 frame_inset 만큼 안쪽에 세운다. 차체가 커지면 -->
+    <!-- 프레임 케이지도 같은 비율로 따라 커진다. 0.20 / 0.34 가 나온다. -->
+    <xacro:property name="frame_inset"  value="0.04"/>   <!-- 차체 옆면 ~ 기둥 바깥면 -->
+    <xacro:property name="post_x"       value="${base_x/2 - frame_inset - post_t/2}"/>  <!-- 기둥 X 위치 -->
+    <xacro:property name="post_y"       value="${base_y/2 - frame_inset - post_t/2}"/>  <!-- 기둥 Y 위치 -->
     <xacro:property name="top_z"        value="${deck_z + frame_h}"/>  <!-- 상단 프레임 z -->
-    <!-- 라이다(하단 상판 전방 중앙) -->
+    <!-- 모터 - 실제 장착 위치. 바퀴 축(x=±wheel_x) 위에서 바퀴 안쪽 면에 -->
+    <!-- 붙어 안쪽(차체 중심 방향)으로 뻗는다. 실물도 모터는 바퀴 안쪽의 -->
+    <!-- 차체 내부에 들어가 있고, 축만 바퀴로 나온다. -->
+    <!-- 차체가 바퀴 바깥면까지 넓어졌으므로 모터는 차체에 완전히 감싸인다. -->
+    <!-- 차체 바닥(z=0) 아래로 나온 아래 절반만 밖에서 보인다. -->
+    <xacro:property name="motor_r"      value="0.04"/>
+    <xacro:property name="motor_len"    value="0.10"/>                           <!-- 모터 몸통 길이 -->
+    <!-- 차체 옆면이 이제 바퀴 안쪽 면과 같은 자리다. 모터 끝면을 거기에 -->
+    <!-- 정확히 맞추면 두 면이 동일 평면이 되어 z-fighting 이 난다. -->
+    <!-- motor_inset 만큼 안으로 물려 확실히 차체 내부에 두자. -->
+    <xacro:property name="motor_inset"  value="0.005"/>
+    <xacro:property name="motor_outer"  value="${wheel_y - wheel_width/2 - motor_inset}"/>
+    <xacro:property name="motor_cy"     value="${motor_outer - motor_len/2}"/>
+    <!-- 센서 장착 위치. 실로봇 TF 라 차체/프레임 모델에 묶지 않는다. -->
+    <!-- 프레임 치수는 미실측 추정이라 여기에 연동시키면 실물이 그대로인데도 -->
+    <!-- 센서 TF 가 따라 움직인다. 실제로 post_x 에 묶었다가 camera_joint 가 -->
+    <!-- 5cm 밀린 적이 있다(2026-08-21). 값은 실측 확보 시에만 바꿀 것. -->
     <xacro:property name="lidar_x"      value="0.16"/>
+    <xacro:property name="camera_x"     value="0.17"/>
     <!-- Materials -->
     <material name="white"><color rgba="0.9 0.9 0.9 1"/></material>
@@ -59,24 +89,23 @@
             <geometry><box size="${base_x} ${base_y} ${base_h}"/></geometry>
         </collision>
-        <!-- 모터 하우징 4개 (빨간 원통). 베이스 하단(z=0)에 부착, 바퀴 안쪽 -->
-        <!-- 모터(y≈±0.19)보다 바퀴(y=±0.25)가 바깥 → 좌우로 돌출 -->
-        <visual>
-            <origin xyz="${wheel_x} ${wheel_y - 0.06} 0" rpy="${pi/2} 0 0"/>
-            <geometry><cylinder radius="0.04" length="0.08"/></geometry>
+        <!-- 모터 하우징 4개 (빨간 원통). 바퀴 축 위, 바퀴 안쪽 면에 직결 -->
+        <visual>
+            <origin xyz="${wheel_x} ${motor_cy} 0" rpy="${pi/2} 0 0"/>
+            <geometry><cylinder radius="${motor_r}" length="${motor_len}"/></geometry>
             <material name="red"/>
         </visual>
         <visual>
-            <origin xyz="${wheel_x} ${-(wheel_y - 0.06)} 0" rpy="${pi/2} 0 0"/>
-            <geometry><cylinder radius="0.04" length="0.08"/></geometry>
+            <origin xyz="${wheel_x} ${-motor_cy} 0" rpy="${pi/2} 0 0"/>
+            <geometry><cylinder radius="${motor_r}" length="${motor_len}"/></geometry>
             <material name="red"/>
         </visual>
         <visual>
-            <origin xyz="${-wheel_x} ${wheel_y - 0.06} 0" rpy="${pi/2} 0 0"/>
-            <geometry><cylinder radius="0.04" length="0.08"/></geometry>
+            <origin xyz="${-wheel_x} ${motor_cy} 0" rpy="${pi/2} 0 0"/>
+            <geometry><cylinder radius="${motor_r}" length="${motor_len}"/></geometry>
             <material name="red"/>
         </visual>
         <visual>
-            <origin xyz="${-wheel_x} ${-(wheel_y - 0.06)} 0" rpy="${pi/2} 0 0"/>
-            <geometry><cylinder radius="0.04" length="0.08"/></geometry>
+            <origin xyz="${-wheel_x} ${-motor_cy} 0" rpy="${pi/2} 0 0"/>
+            <geometry><cylinder radius="${motor_r}" length="${motor_len}"/></geometry>
             <material name="red"/>
         </visual>
@@ -348,6 +377,9 @@
         <parent link="frame"/>
         <child link="camera_link"/>
-        <!-- 상단 전면 가로 프로파일(z=deck_z+0.32)에 부착. 전방(+X) 주시 -->
-        <origin xyz="${post_x + 0.02} 0 ${deck_z + 0.32}" rpy="0 0 0"/>
+        <!-- 상단 전면 가로 프로파일(z=deck_z+0.32) 높이. 전방(+X) 주시 -->
+        <!-- x 는 camera_x 고정값이다. post_x 에 묶으면 프레임 모델을 손댈 때마다 -->
+        <!-- 실로봇 TF 가 흔들린다. 프레임 가로바가 이보다 조금 앞에 있어 -->
+        <!-- 비주얼상 7mm 정도 떠 보이지만, TF 안정성이 우선이다. -->
+        <origin xyz="${camera_x} 0 ${deck_z + 0.32}" rpy="0 0 0"/>
     </joint>
     <!-- 광학 프레임 (ROS optical 규약 - z 전방, x 우측, y 하방) -->
